Commit message: upload

File: l6/urdf/xacro/gazebo/mbot_base_gazebo.xacro (robot description, xacro)
@@ -12,5 +12,5 @@
     <xacro:property name="wheel_joint_z" value="0.05"/>
     <xacro:property name="caster_mass"    value="0.5" />
-    <xacro:property name="caster_radius" value="0.015"/> <!-- (wheel_radius - ( base_length/2 - wheel_joint_z))/2 -->
+    <xacro:property name="caster_radius"  value="0.015"/> <!-- wheel_radius - ( base_length/2 - wheel_joint_z) -->
     <xacro:property name="caster_joint_x" value="0.18"/>
     <!-- Defining the colors used in this robot -->
@@ -25,4 +25,12 @@
     </material>
     <!-- Macro for inertia matrix -->
+    <xacro:macro name="sphere_inertial_matrix" params="m r">
+        <inertial>
+            <mass value="${m}" />
+            <inertia ixx="${2*m*r*r/5}" ixy="0" ixz="0"
+                iyy="${2*m*r*r/5}" iyz="0"
+                izz="${2*m*r*r/5}" />
+        </inertial>
+    </xacro:macro>
     <xacro:macro name="cylinder_inertial_matrix" params="m r h">
         <inertial>
@@ -31,12 +39,4 @@
                 iyy="${m*(3*r*r+h*h)/12}" iyz = "0"
                 izz="${m*r*r/2}" />
-        </inertial>
-    </xacro:macro>
-    <xacro:macro name="sphere_inertial_matrix" params="m r">
-        <inertial>
-            <mass value="${m}" />
-            <inertia ixx="${2*m*r*r/5}" ixy="0" ixz="0"
-                iyy="${2*m*r*r/5}" iyz="0"
-                izz="${2*m*r*r/5}" />
         </inertial>
     </xacro:macro>
@@ -57,5 +57,5 @@
                 <material name="gray" />
             </visual>
-	    <collision>
+            <collision>
                 <origin xyz="0 0 0" rpy="${M_PI/2} 0 0" />
                 <geometry>
@@ -65,8 +65,8 @@
             <cylinder_inertial_matrix  m="${wheel_mass}" r="${wheel_radius}" h="${wheel_length}" />
         </link>
-	<gazebo reference="${prefix}_wheel_link">
+        <gazebo reference="${prefix}_wheel_link">
             <material>Gazebo/Gray</material>
         </gazebo>
-	<!-- Transmission is important to link the joints and the controller -->
+        <!-- Transmission is important to link the joints and the controller -->
         <transmission name="${prefix}_wheel_joint_trans">
             <type>transmission_interface/SimpleTransmission</type>
@@ -96,5 +96,5 @@
                 <material name="black" />
             </visual>
-	    <collision>
+            <collision>
                 <origin xyz="0 0 0" rpy="0 0 0"/>
                 <geometry>
@@ -104,6 +104,9 @@
             <sphere_inertial_matrix  m="${caster_mass}" r="${caster_radius}" />
         </link>
+        <gazebo reference="${prefix}_caster_link">
+            <material>Gazebo/Black</material>
+        </gazebo>
     </xacro:macro>
-    <xacro:macro name="mbot_base">
+    <xacro:macro name="mbot_base_gazebo">
         <link name="base_footprint">
             <visual>
@@ -114,5 +117,5 @@
             </visual>
         </link>
-	<gazebo reference="base_footprint">
+        <gazebo reference="base_footprint">
             <turnGravityOff>false</turnGravityOff>
         </gazebo>
@@ -130,5 +133,5 @@
                 <material name="yellow" />
             </visual>
-	    <collision>
+            <collision>
                 <origin xyz=" 0 0 0" rpy="0 0 0" />
                 <geometry>
@@ -138,12 +141,12 @@
             <cylinder_inertial_matrix  m="${base_mass}" r="${base_radius}" h="${base_length}" />
         </link>
-	<gazebo reference="base_link">
+        <gazebo reference="base_link">
             <material>Gazebo/Blue</material>
         </gazebo>
-        <wheel prefix="left" reflect="-1"/>
+        <wheel prefix="left"  reflect="-1"/>
         <wheel prefix="right" reflect="1"/>
         <caster prefix="front" reflect="-1"/>
-        <caster prefix="back" reflect="1"/>
-	<!-- controller -->
+        <caster prefix="back"  reflect="1"/>
+        <!-- controller -->
         <gazebo>
             <plugin name="differential_drive_controller"
